File: AudioMixer/AudioMixer.kicad_sch (KiCad schematic)
At the start: 44 parts, among them U1 NJM4580, U2 NJM4580, U3 NJM4580, U4 NJM4580

Commit message: Update comment
Other:
- note added: "減衰アンプ : 0.2695 (-11.39dB) 前段の最大出力を21Vp-pとしたとき LINE OUTの標準である2V RMSに収まるようにする。"
- note removed: "減衰アンプ : 0.28 (-11.1dB) 前段の最大出力を20Vp-pとしたとき LINE OUTの標準である2V RMSに収まるようにする。 Input : 20Vp-p(max) Output : 5.6Vp-p (2V RMS : Audio LINE OUT) 0.28 = 10K / (33K + 2.2K)"
Changed lines of the file:
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@@
 		)
 	)
-	(text "減衰アンプ : 0.28 (-11.1dB)\n前段の最大出力を20Vp-pとしたとき\nLINE OUTの標準である2V RMSに収まるようにする。\n\nInput : 20Vp-p(max)\nOutput : 5.6Vp-p (2V RMS : Audio LINE OUT)\n0.28 = 10K / (33K + 2.2K)"
+	(text "減衰アンプ : 0.2695 (-11.39dB)\n前段の最大出力を21Vp-pとしたとき\nLINE OUTの標準である2V RMSに収まるようにする。"
 		(exclude_from_sim no)
-		(at 150.114 83.058 0)
+		(at 150.368 81.534 0)
 		(effects
 			(font
